File: output.kicad_pcb (KiCad board)
At the start: 2 copper layers, 90 x 90 mm, 2 parts

Commit message: Add files via upload
Parts:
- added #PWR03: svg:vias, svg:vias, F.Cu at (0.00, 0.00)
Routing:
- net ffd42a: vias 1 -> 0
Changed lines of the file:
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@@
 	(version 20231120)
 	(generator "svg2kicad")
-	(generator_version "1.0-mvp")
+	(generator_version "1.0.1")
 	(general
 		(thickness 1.6)
@@
 		(property "Reference" "#PWR01" (at 0 0 0) (layer "F.SilkS") (effects (font (size 1 1) (thickness 0.15)) hide))
 		(property "Value" "svg:converted-F" (at 0 0 0) (layer "F.Fab") (effects (font (size 1 1) (thickness 0.15))))
-		(pad "1" thru_hole circle (at 30.874996 36.324779) (size 2.887101 2.887101) (drill 1.698197) (layers "*.Cu" "*.Mask") (net 1 "ffd42a"))
+		(pad "1" thru_hole circle (at 41.310933 42.533502) (size 2.887101 2.887101) (drill 1.698197) (layers "*.Cu" "*.Mask") (net 1 "ffd42a"))
 		(pad "2" thru_hole circle (at 85.08372 49.318899) (size 2.887101 2.887101) (drill 1.698197) (layers "*.Cu" "*.Mask") (net 2 "ff00ff"))
 		(pad "3" smd circle (at 62.008371 28.826287) (size 2.887101 2.887101) (layers "F.Cu" "F.Paste" "F.Mask") (net 2 "ff00ff"))
 		(pad "4" smd circle (at 64.941127 62.117311) (size 2.887101 2.887101) (layers "F.Cu" "F.Paste" "F.Mask") (net 2 "ff00ff"))
+		(pad "5" smd circle (at 21.810429 49.418661) (size 2.887101 2.887101) (layers "F.Cu" "F.Paste" "F.Mask") (net 1 "ffd42a"))
 	)
 	(footprint "svg:converted-B"
@@
 		(property "Reference" "#PWR02" (at 0 0 0) (layer "F.SilkS") (effects (font (size 1 1) (thickness 0.15)) hide))
 		(property "Value" "svg:converted-B" (at 0 0 0) (layer "F.Fab") (effects (font (size 1 1) (thickness 0.15))))
-		(pad "1" smd circle (at 34.022579 85.111796) (size 2.887101 2.887101) (layers "B.Cu" "B.Paste" "B.Mask") (net 1 "ffd42a"))
+		(pad "1" smd circle (at 25.436049 91.584715) (size 2.887101 2.887101) (layers "B.Cu" "B.Paste" "B.Mask") (net 1 "ffd42a"))
 	)
-	(via (at 45.286526 71.030497) (size 1.494014) (drill 0.896409) (layers "F.Cu" "B.Cu") (net 1))
+	(footprint "svg:vias"
+		(layer "F.Cu")
+		(at 0 0)
+		(property "Reference" "#PWR03" (at 0 0 0) (layer "F.SilkS") (effects (font (size 1 1) (thickness 0.15)) hide))
+		(property "Value" "svg:vias" (at 0 0 0) (layer "F.Fab") (effects (font (size 1 1) (thickness 0.15))))
+		(pad "V1" thru_hole circle (at 32.244595 67.119126) (size 0.471699 0.471699) (drill 0.283019) (layers "*.Cu" "*.Mask") (net 1 "ffd42a"))
+	)
 	(zone
 		(net 0)
@@
 		(polygon
 			(pts
-				(xy 70.734028 44.522777)
-				(xy 71.717832 30.425335)
-				(xy 84.667593 38.247906)
+				(xy 73.640238 48.882093)
+				(xy 74.624042 34.78465)
+				(xy 87.573803 42.607222)
 			)
 		)
